File: faceplates/D32 Joystick Adapter Faceplate A1/D32 Joystick Adapter Faceplate A1.kicad_pcb (KiCad board)
At the start: 2 copper layers, 48.9 x 40.6 mm, 5 parts, among them M1 Mounting, M2 Mounting, M3 Mounting, M4 Mounting

Commit message: Changed faceplate cutout
Parts:
- moved G*** 0.58 mm to (123.1, 94.7)
Other:
- outline, holes or cut-outs redrawn
